Commit message: Revise TALON-6 as asymmetrical five-digit right hand

File: assets/models/studio/sources/talon6/hand.urdf (robot description, URDF)
Before this commit: robot TALON-6-dual-opposition, 7 links, 6 joints
Links:
- removed link radial_thumb_digit
- removed link ulnar_thumb_digit
- added link thumb_digit; visual mesh filename=meshes/thumb.obj; visual mesh filename=meshes/thumb_pad.obj
- added link thumb_hub; visual mesh filename=meshes/motor_cap.obj; visual mesh filename=meshes/motor_cover.obj
- link palm: geometry visual mesh filename=meshes/motor_cap.obj; visual mesh filename=meshes/motor_cap.obj
Joints:
- removed joint radial_thumb_flex
- removed joint ulnar_thumb_flex
- added joint thumb_flex: type revolute, parent thumb_hub, child thumb_digit, origin xyz=0 0 0 rpy=0.2617993877991494 0 0, axis -1 0 0, limit lower=0 upper=1.4835298641951802 effort=1.5 velocity=2.0
- added joint thumb_opposition: type revolute, parent palm, child thumb_hub, origin xyz=0.075 0.027 0.065 rpy=0 0 1.2217304763960306, axis 0 0 1, limit lower=-0.3490658503988659 upper=0.6108652381980153 effort=1.5 velocity=2.0
