Commit message: Refine hand studio display assets and Wuji motor bands

File: assets/models/studio/sources/talon9/hand.urdf (robot description, URDF)
Before this commit: robot TALON-9-right-hand, 10 links, 9 joints
Links:
- link index_distal: geometry visual mesh filename=meshes/distal_pad.obj scale=0.82 0.82 0.82; visual mesh filename=meshes/distal_shell.obj scale=0.82 0.82 0.82
- link index_proximal: geometry visual mesh filename=meshes/motor_cap.obj scale=0.82 0.82 0.82; visual mesh filename=meshes/motor_cover.obj scale=0.82 0.82 0.82
- link middle_distal: geometry visual mesh filename=meshes/distal_pad.obj scale=0.82 0.82 0.82; visual mesh filename=meshes/distal_shell.obj scale=0.82 0.82 0.82
- link middle_proximal: geometry visual mesh filename=meshes/motor_cap.obj scale=0.82 0.82 0.82; visual mesh filename=meshes/motor_cover.obj scale=0.82 0.82 0.82
- link palm: geometry visual mesh filename=meshes/motor_cover.obj scale=0.82 0.82 0.82; visual mesh filename=meshes/motor_cover.obj scale=0.82 0.82 0.82
- link ring_distal: geometry visual mesh filename=meshes/distal_pad.obj scale=0.82 0.82 0.82; visual mesh filename=meshes/distal_shell.obj scale=0.82 0.82 0.82
- link ring_proximal: geometry visual mesh filename=meshes/motor_cap.obj scale=0.82 0.82 0.82; visual mesh filename=meshes/motor_cover.obj scale=0.82 0.82 0.82
- link thumb_base_hub: geometry visual mesh filename=meshes/motor_cap.obj scale=0.86 0.86 0.86; visual mesh filename=meshes/motor_cover.obj scale=0.75 0.75 0.75
- link thumb_distal: geometry visual mesh filename=meshes/distal_pad.obj scale=0.66 0.66 0.561; visual mesh filename=meshes/distal_shell.obj scale=0.66 0.66 0.561
- link thumb_proximal: geometry visual mesh filename=meshes/motor_cap.obj scale=0.68 0.68 0.68; visual mesh filename=meshes/motor_cover.obj scale=0.68 0.68 0.68
Joints:
- joint index_mcp_flex: origin xyz=0.027 0 0.048 rpy=0 0 0 -> xyz=0.027 0.003 0.048 rpy=0 0 0
- joint index_pip_flex: origin xyz=0 0 0.047 rpy=0 0 0 -> xyz=0 0 0.03948 rpy=0 0 0
- joint middle_mcp_flex: origin xyz=0.008 0 0.048 rpy=0 0 0 -> xyz=0.008 0.003 0.048 rpy=0 0 0
- joint middle_pip_flex: origin xyz=0 0 0.047 rpy=0 0 0 -> xyz=0 0 0.03948 rpy=0 0 0
- joint ring_mcp_flex: origin xyz=-0.011 0 0.048 rpy=0 0 0 -> xyz=-0.011 0.003 0.048 rpy=0 0 0
- joint ring_pip_flex: origin xyz=0 0 0.047 rpy=0 0 0 -> xyz=0 0 0.03948 rpy=0 0 0
- joint thumb_base_sweep: axis 0 1 0 -> 0 0 1; limit lower=-0.5235987755982988 upper=0.5235987755982988 effort=1.5 velocity=2.0 -> lower=-0.3490658503988659 upper=1.5009831567151235 effort=1.5 velocity=2.0; origin xyz=0.043 0.025 0.057 rpy=0 -0.8726646259971648 0 -> xyz=0.018 0.024 0.023 rpy=0 0 0
- joint thumb_mcp_flex: origin xyz=0 0 0 rpy=0 0 0 -> xyz=0.031 0.017 0.011 rpy=0 0 0
- joint thumb_pip_flex: origin xyz=0 0 0.04042 rpy=0 0 0 -> xyz=0 0 0.034 rpy=0 0 0

Commit message: Refine TALON teaser and poses; close MIDAS preview linkages

File: assets/models/studio/sources/talon9/hand.urdf (robot description, URDF)
Before this commit: robot TALON-9-right-hand, 10 links, 9 joints
Links:
- link thumb_base_hub: geometry visual mesh filename=meshes/motor_cap.obj scale=0.86 0.86 0.86; visual mesh filename=meshes/motor_cover.obj scale=0.82 0.82 0.82
- link thumb_distal: geometry visual mesh filename=meshes/distal_pad.obj scale=0.82 0.82 0.82; visual mesh filename=meshes/distal_shell.obj scale=0.82 0.82 0.82
- link thumb_proximal: geometry visual mesh filename=meshes/motor_cap.obj scale=0.82 0.82 0.82; visual mesh filename=meshes/motor_cover.obj scale=0.82 0.82 0.82
Joints:
- joint thumb_base_sweep: origin xyz=0.018 0.024 0.023 rpy=0 0 0 -> xyz=0.018 0.014 0.011 rpy=0 0 0
- joint thumb_mcp_flex: origin xyz=0.031 0.017 0.011 rpy=0 0 0 -> xyz=0.029 0.014 0.011 rpy=0 0 0
- joint thumb_pip_flex: origin xyz=0 0 0.034 rpy=0 0 0 -> xyz=0 0 0.03948 rpy=0 0 0
